File: MainBoard/MainBoard.sch (KiCad schematic (older format))
At the start: 16 parts

Commit message: add PV supply circuit
Connections:
- wire segments 29 -> 32
Other:
- moved on the sheet: U?
Changed lines of the file:
@@
 L Sensor_Motion:LSM9DS1 U?
 U 1 1 605F11C5
-P 7350 1400
-F 0 "U?" H 7350 511 50  0000 C CNN
-F 1 "LSM9DS1" H 7350 420 50  0000 C CNN
-F 2 "Package_LGA:LGA-24L_3x3.5mm_P0.43mm" H 8850 2150 50  0001 C CNN
-F 3 "http://www.st.com/content/ccc/resource/technical/document/datasheet/1e/3f/2a/d6/25/eb/48/46/DM00103319.pdf/files/DM00103319.pdf/jcr:content/translations/en.DM00103319.pdf" H 7350 1500 50  0001 C CNN
-	1    7350 1400
-	1    0    0    -1
-$EndComp
-Text GLabel 6650 1000 0    50   Input ~ 0
+P 7100 1500
+F 0 "U?" H 7100 611 50  0000 C CNN
+F 1 "LSM9DS1" H 7100 520 50  0000 C CNN
+F 2 "Package_LGA:LGA-24L_3x3.5mm_P0.43mm" H 8600 2250 50  0001 C CNN
+F 3 "http://www.st.com/content/ccc/resource/technical/document/datasheet/1e/3f/2a/d6/25/eb/48/46/DM00103319.pdf/files/DM00103319.pdf/jcr:content/translations/en.DM00103319.pdf" H 7100 1600 50  0001 C CNN
+	1    7100 1500
+	1    0    0    -1
+$EndComp
+Text GLabel 6400 1100 0    50   Input ~ 0
 SCL
-Text GLabel 6650 1100 0    50   Input ~ 0
+Text GLabel 6400 1200 0    50   Input ~ 0
 SDA
 Text GLabel 1350 5950 0    50   Input ~ 0
@@
 L Connector:Micro_SD_Card J?
 U 1 1 605FDC7D
-P 10250 1600
-F 0 "J?" H 10200 2317 50  0000 C CNN
-F 1 "Micro_SD_Card" H 10200 2226 50  0000 C CNN
-F 2 "" H 11400 1900 50  0001 C CNN
-F 3 "http://katalog.we-online.de/em/datasheet/693072010801.pdf" H 10250 1600 50  0001 C CNN
-	1    10250 1600
+P 10300 2450
+F 0 "J?" H 10250 3167 50  0000 C CNN
+F 1 "Micro_SD_Card" H 10250 3076 50  0000 C CNN
+F 2 "" H 11450 2750 50  0001 C CNN
+F 3 "http://katalog.we-online.de/em/datasheet/693072010801.pdf" H 10300 2450 50  0001 C CNN
+	1    10300 2450
 	1    0    0    -1
 $EndComp
@@
 L power:GND #PWR?
 U 1 1 605FFED7
-P 7250 2200
-F 0 "#PWR?" H 7250 1950 50  0001 C CNN
-F 1 "GND" H 7255 2027 50  0000 C CNN
-F 2 "" H 7250 2200 50  0001 C CNN
-F 3 "" H 7250 2200 50  0001 C CNN
-	1    7250 2200
-	1    0    0    -1
+P 7000 2300
+F 0 "#PWR?" H 7000 2050 50  0001 C CNN
+F 1 "GND" H 7005 2127 50  0000 C CNN
+F 2 "" H 7000 2300 50  0001 C CNN
+F 3 "" H 7000 2300 50  0001 C CNN
+	1    7000 2300
+	0    1    1    0
 $EndComp
 $Comp
 L power:GND #PWR?
 U 1 1 60600088
-P 7450 2200
-F 0 "#PWR?" H 7450 1950 50  0001 C CNN
-F 1 "GND" H 7455 2027 50  0000 C CNN
-F 2 "" H 7450 2200 50  0001 C CNN
-F 3 "" H 7450 2200 50  0001 C CNN
-	1    7450 2200
-	1    0    0    -1
+P 7200 2300
+F 0 "#PWR?" H 7200 2050 50  0001 C CNN
+F 1 "GND" H 7205 2127 50  0000 C CNN
+F 2 "" H 7200 2300 50  0001 C CNN
+F 3 "" H 7200 2300 50  0001 C CNN
+	1    7200 2300
+	0    -1   -1   0
 $EndComp
 $Comp
 L power:GND #PWR?
 U 1 1 60600A3A
-P 11050 2200
-F 0 "#PWR?" H 11050 1950 50  0001 C CNN
-F 1 "GND" H 11055 2027 50  0000 C CNN
-F 2 "" H 11050 2200 50  0001 C CNN
-F 3 "" H 11050 2200 50  0001 C CNN
-	1    11050 2200
+P 11100 3050
+F 0 "#PWR?" H 11100 2800 50  0001 C CNN
+F 1 "GND" H 11105 2877 50  0000 C CNN
+F 2 "" H 11100 3050 50  0001 C CNN
+F 3 "" H 11100 3050 50  0001 C CNN
+	1    11100 3050
 	1    0    0    -1
 $EndComp
@@
 Wire Wire Line
 	9700 5750 9500 5750
+$Comp
+L power:+3.3V #PWR?
+U 1 1 60630579
+P 7400 700
+F 0 "#PWR?" H 7400 550 50  0001 C CNN
+F 1 "+3.3V" H 7415 873 50  0000 C CNN
+F 2 "" H 7400 700 50  0001 C CNN
+F 3 "" H 7400 700 50  0001 C CNN
+	1    7400 700
+	1    0    0    -1
+$EndComp
+Wire Wire Line
+	7500 700  7400 700
+Connection ~ 7200 700
+Wire Wire Line
+	7200 700  7100 700
+Connection ~ 7400 700
+Wire Wire Line
+	7400 700  7200 700
 $EndSCHEMATC

Commit message: add final sensors and update PCB
Parts:
- removed U?: STM32L031K6Tx, Package_QFP:LQFP-32_7x7mm_P0.8mm, symbol MCU_ST_STM32L0:STM32L031K6Tx
- added TP1: PWR-REGLP2S, TestPoint:TestPoint_Pad_4.0x4.0mm, symbol Connector:TestPoint
- added TP2: JTRST, TestPoint:TestPoint_Pad_4.0x4.0mm, symbol Connector:TestPoint
- added TP3: PWR-REGLP1S, TestPoint:TestPoint_Pad_4.0x4.0mm, symbol Connector:TestPoint
- added TP4: JTO-SWO, TestPoint:TestPoint_Pad_4.0x4.0mm, symbol Connector:TestPoint
- added TP5: RF-NRST, TestPoint:TestPoint_Pad_4.0x4.0mm, symbol Connector:TestPoint
- added TP6: RF-SMPSRDY, TestPoint:TestPoint_Pad_4.0x4.0mm, symbol Connector:TestPoint
- added TP7: JTCK-SWDIO, TestPoint:TestPoint_Pad_4.0x4.0mm, symbol Connector:TestPoint
- added TP8: JTMS-SWDIO, TestPoint:TestPoint_Pad_4.0x4.0mm, symbol Connector:TestPoint
- added TP9: JTO-SWCLK, TestPoint:TestPoint_Pad_4.0x4.0mm, symbol Connector:TestPoint
- added U3: STM32WL55CCU7, libs:STM32WL55CCU7, symbol STM32WL55CCU7:STM32WL55CCU7
- C1, C2: renamed from C?; footprint (none) -> Capacitor_SMD:C_0805_2012Metric_Pad1.18x1.45mm_HandSolder
- J1: renamed from J?; footprint (none) -> Connector_PinHeader_1.00mm:PinHeader_1x02_P1.00mm_Horizontal
- J2: renamed from J?; footprint (none) -> Connector_Card:microSD_HC_Hirose_DM3AT-SF-PEJM5
- J3: renamed from J?; footprint (none) -> Connector_USB:USB_C_Receptacle_Amphenol_12401548E4-2A
- JP1: renamed from JP?; footprint (none) -> Jumper:SolderJumper-2_P1.3mm_Open_RoundedPad1.0x1.5mm
- L1: renamed from L?; footprint (none) -> Inductor_THT:L_Axial_L5.0mm_D3.6mm_P10.00mm_Horizontal_Murata_BL01RN1A2A2
- R1, R2: renamed from R?; footprint (none) -> Resistor_SMD:R_0805_2012Metric
- gave numbers to parts that had none: 6
Connections:
- net labels added: RX, TX
- wire segments 32 -> 39

Commit message: lots of work on PCB
Parts:
- removed D1: Inolux_IN-PI554FCH, LED_SMD:LED_Inolux_IN-PI554FCH_PLCC4_5.0x5.0mm_P3.2mm, symbol LED:Inolux_IN-PI554FCH
- removed J2: Micro_SD_Card, Connector_Card:microSD_HC_Hirose_DM3AT-SF-PEJM5, symbol Connector:Micro_SD_Card
- removed J3: USB_C_Receptacle, Connector_USB:USB_C_Receptacle_Amphenol_12401548E4-2A, symbol Connector:USB_C_Receptacle
- removed U1: MAX-8C, RF_GPS:ublox_MAX, symbol RF_GPS:MAX-8C
- removed U5: FUSB302B01MPX, Package_DFN_QFN:WQFN-14-1EP_2.5x2.5mm_P0.5mm_EP1.45x1.45mm, symbol Interface_USB:FUSB302B01MPX
- added BT1: Battery_Cell, Connector_PinHeader_1.00mm:PinHeader_1x02_P1.00mm_Horizontal, symbol Device:Battery_Cell
- added C10, C11, C12, C13, C15, C16, C17, C18, C19, C20, C21, C22, C23, C24, C25, C26, C27, C28, C29, C30, C31, C32, C33, C34, C35, C5, C8, C9: 0.1uF, Capacitor_SMD:C_0402_1005Metric, symbol Device:C_Small
- added C14: 2.2uF, Capacitor_SMD:C_0402_1005Metric, symbol Device:C_Small
- added C3, C7: 4.7uF, Capacitor_SMD:C_0402_1005Metric, symbol Device:C_Small
- added C36, C37, C38, C39, C40, C41, C42, C43, C44, C45, C46, C47, C48, C49, C50, C51, C52: _, Capacitor_SMD:C_0402_1005Metric, symbol Device:C_Small
- added C4: 10uF, Capacitor_SMD:C_0402_1005Metric, symbol Device:C_Small
- added C6: 1uF, Capacitor_SMD:C_0402_1005Metric, symbol Device:C_Small
- added D1: DIODE, Diode_SMD:D_0402_1005Metric, symbol pspice:DIODE
- added IC2: TESEO-LIV3F, libs:SON110P970X1010X230-18N, symbol TESEO-LIV3F:TESEO-LIV3F
- added J2, J7: Conn_Coaxial, Connector_Coaxial:U.FL_Hirose_U.FL-R-SMT-1_Vertical, symbol Connector:Conn_Coaxial
- added J3: Conn_01x30_Female, libs:waveshare_1.02, symbol Connector:Conn_01x30_Female
- added J4, J5: RX, Connector_Coaxial:U.FL_Hirose_U.FL-R-SMT-1_Vertical, symbol Connector:Conn_Coaxial
- added J6: Conn_01x04, libs:4 Pin SMD Wire, symbol Connector_Generic:Conn_01x04
- added JP2: BAT EN, Jumper:SolderJumper-2_P1.3mm_Open_RoundedPad1.0x1.5mm, symbol Jumper:SolderJumper_2_Open
- added L10, L11, L12: _, Inductor_SMD:L_0402_1005Metric, symbol pspice:INDUCTOR
- added L2: 1uH, Inductor_SMD:L_Coilcraft_LPS4018, symbol pspice:INDUCTOR
- added L3, L4, L5, L6, L7, L8, L9: 1uH, Inductor_SMD:L_0402_1005Metric, symbol pspice:INDUCTOR
- added R3, R4, R5: R_US, Resistor_SMD:R_0402_1005Metric, symbol Device:R_US
- added SW1, SW2, SW3: SW_DIP_x01, Button_Switch_SMD:SW_Push_1P1T-SH_NO_CK_KMR2xxG, symbol Switch:SW_DIP_x01
- added TP10: GND, TestPoint:TestPoint_Pad_2.0x2.0mm, symbol Connector:TestPoint
- added TP11: BATT, TestPoint:TestPoint_Pad_2.0x2.0mm, symbol Connector:TestPoint
- added TP12: RX, TestPoint:TestPoint_Pad_2.0x2.0mm, symbol Connector:TestPoint
- added TP13: TX, TestPoint:TestPoint_Pad_2.0x2.0mm, symbol Connector:TestPoint
- added TP14: 3.3V, TestPoint:TestPoint_Pad_2.0x2.0mm, symbol Connector:TestPoint
- added TP15: BLE RSTN, TestPoint:TestPoint_Pad_2.0x2.0mm, symbol Connector:TestPoint
- added U1: BLUENRG-355MC, libs:BLUENRG, symbol BLUENRG:BLUENRG-355MC
- added U6: ADP2108AUJ-3.3, Package_TO_SOT_SMD:TSOT-23-5, symbol Regulator_Switching:ADP2108AUJ-3.3
- added Y1, Y2, Y3, Y4: Crystal, Crystal:Crystal_SMD_2012-2Pin_2.0x1.2mm, symbol Device:Crystal
- C1, C2: footprint Capacitor_SMD:C_0805_2012Metric_Pad1.18x1.45mm_HandSolder -> Capacitor_SMD:C_0402_1005Metric
- L1: footprint Inductor_THT:L_Axial_L5.0mm_D3.6mm_P10.00mm_Horizontal_Murata_BL01RN1A2A2 -> Inductor_SMD:L_Coilcraft_LPS4018
- R1, R2: footprint Resistor_SMD:R_0805_2012Metric -> Resistor_SMD:R_0402_1005Metric
- TP1: value PWR-REGLP2S -> NRST; footprint TestPoint:TestPoint_Pad_4.0x4.0mm -> TestPoint:TestPoint_Pad_2.0x2.0mm
- TP2, TP4, TP7, TP8, TP9: footprint TestPoint:TestPoint_Pad_4.0x4.0mm -> TestPoint:TestPoint_Pad_2.0x2.0mm
- TP3: value PWR-REGLP1S -> BLE TX; footprint TestPoint:TestPoint_Pad_4.0x4.0mm -> TestPoint:TestPoint_Pad_2.0x2.0mm
- TP5: value RF-NRST -> PA10; footprint TestPoint:TestPoint_Pad_4.0x4.0mm -> TestPoint:TestPoint_Pad_2.0x2.0mm
- TP6: value RF-SMPSRDY -> BLE RX; footprint TestPoint:TestPoint_Pad_4.0x4.0mm -> TestPoint:TestPoint_Pad_2.0x2.0mm
Connections:
- net labels added: RFI_N, RFI_P, RFO_HP, RX1, SPI1-MISO, SPI1-MOSI, SPI1-SCK, TX1, VR_PA
- wire segments 39 -> 193
Other:
- note added: "BLE\n\n"
- note added: "DISPLAY\n"
- note added: "GPS\n"
- note added: "HR"
- note added: "IMU\n"
- note added: "LoRa + main uC\n"
- note added: "LoRa RF\n"
- note added: "POWER\n"
- moved on the sheet: C1, C2, IC1, J1, JP1, L1, R1, R2, TP2, TP4, TP7, TP8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

Commit message: lots of work on PCB
Parts:
- removed C36: _, Capacitor_SMD:C_0402_1005Metric, symbol Device:C_Small
- removed C4: 10uF, Capacitor_SMD:C_0402_1005Metric, symbol Device:C_Small
- removed JP2: BAT EN, Jumper:SolderJumper-2_P1.3mm_Open_RoundedPad1.0x1.5mm, symbol Jumper:SolderJumper_2_Open
- removed L2: 1uH, Inductor_SMD:L_Coilcraft_LPS4018, symbol pspice:INDUCTOR
- removed R1: SET R1, Resistor_SMD:R_0402_1005Metric, symbol Device:R_Small_US
- removed R2: SET R2, Resistor_SMD:R_0402_1005Metric, symbol Device:R_Small_US
- removed U2: TPS61201DRC, Package_SON:Texas_S-PVSON-N10_ThermalVias, symbol Regulator_Switching:TPS61201DRC
- removed U6: ADP2108AUJ-3.3, Package_TO_SOT_SMD:TSOT-23-5, symbol Regulator_Switching:ADP2108AUJ-3.3
- added C?: 0.1uF, Capacitor_SMD:C_0402_1005Metric, symbol Device:C_Small
- added C? (x3): 10uF, Capacitor_SMD:C_0402_1005Metric, symbol Device:C_Small
- added C?: 10nF, Capacitor_SMD:C_0402_1005Metric, symbol Device:C_Small
- added C?: 100uF, Capacitor_SMD:C_0402_1005Metric, symbol Device:C_Small
- added D?: 1.8V, symbol Device:D_Zener
- added L?: 1uH, Inductor_SMD:L_0402_1005Metric, symbol pspice:INDUCTOR
- added R1: 5K, Resistor_SMD:R_0402_1005Metric, symbol Device:R_US
- added R2: R_US, Resistor_SMD:R_0402_1005Metric, symbol Device:R_US
- added R?: 100, Resistor_SMD:R_0402_1005Metric, symbol Device:R_US
- added TH1: Thermistor, symbol Device:Thermistor
- added U2: MAX20361AEWC+, libs:MAX20361AEWC&plus_, symbol MAX2036:MAX20361AEWC+
- added U?: TPS63001, Package_SON:Texas_DRC0010J_ThermalVias, symbol Regulator_Switching:TPS63001
- C1: value 10uF -> 1uF
- C2: value 0.1uF -> 1uF
- C3: value 4.7uF -> 1uF
- L1: value 2.2uH -> INDUCTOR; footprint Inductor_SMD:L_Coilcraft_LPS4018 -> Inductor_SMD:L_0402_1005Metric
Connections:
- net +3V3: now also IC1.10 (VLED+), IC1.9 (VLED+), U4.13 (DEN_A/G), U4.7 (CS_A/G), U4.8 (CS_M), C?.1, C?.1, D?.1 (K), U?.1 (VOUT), U?.10 (FB); no longer C3.2, U3.11 (VDD), U3.25 (VDDPA), U3.28 (VDDRF), U3.44 (VDD)
- net GND: now also C2.2, C3.2, U4.14 (RES), U4.15 (RES), U4.16 (RES), U4.17 (RES), U4.18 (RES), U4.5 (SDO_A/G), U4.6 (SDO_M), C?.2, C?.2, C?.2, C?.2, C?.2, C?.2, R1.1, TH1.1, U2.B2 (GND), U?.11 (PGND), U?.3 (PGND), U?.9 (GND); no longer C2.1
- net SCL: now also U2.A4 (SCL)
- net SDA: now also U2.A3 (SDA)
- net at BT1.1 (+), JP1.2 (B), TP11.1: now also U?.5 (VIN); no longer C3.1
- net at IC1.11 (VDD): now also D?.2 (A)
- net at JP1.1 (A): now also C3.1, U2.C2 (SYS)
- net at L1.2: now also U2.B1 (SRC)
- net at J1.2 (Pin_2), L1.1: now also U2.C1 (LX); no longer C1.1
- net at U4.21 (CAP): now also C?.1
- net at U4.24 (C1): now also C?.1
- new net: R1.2, U2.A1 (*EN)
- new net: R2.2, U2.B4 (REF)
- new net: C2.1, U2.C3 (VCC)
- new net: R2.1, TH1.2, U2.C4 (THM)
- new net: L?.2, U?.2 (L2)
- new net: L?.1, U?.4 (L1)
- new net: C?.1, R?.2, U?.6 (EN), U?.7 (PS/SYNC), U?.8 (VINA)
Other:
- moved on the sheet: BT1, J1, JP1, TP11

Commit message: clean silkscreen, add power delivery, route LoRa RF
Parts:
- added C?: _, Capacitor_SMD:C_0402_1005Metric, symbol Device:C_Small
- added JP?: PV EN, Jumper:SolderJumper-2_P1.3mm_Open_RoundedPad1.0x1.5mm, symbol Jumper:SolderJumper_2_Open
- gave numbers to parts that had none: 10
Connections:
- net +3V3: now also U3.11 (VDD), U3.28 (VDDRF), U3.37 (VBAT), U3.41 (VDDA), U3.44 (VDD), U3.46 (VDDSMPS)
- net GND: now also U3.48 (VSSSMPS), C?.1
- net at BT1.1 (+), JP1.2 (B), TP11.1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: now also C53.1, R6.1
- net at J1.2 (Pin_2), L1.1, U2.C1 (LX): now also C1.1
- net at U3.19 (PH3-BOOT0): now also JP?.2 (B)
- net at U3.25 (VDDPA): now also U3.29 (VDDRF1V55), U3.45 (VFBSMPS), C?.2

Commit message: add pdfs
Parts:
- gave numbers to parts that had none: 2
Changed lines of the file:
@@
 Connection ~ 1800 2050
 $Comp
-L power:GND #PWR?
+L power:GND #PWR0125
 U 1 1 61D11080
 P 9000 5650
-F 0 "#PWR?" H 9000 5400 50  0001 C CNN
+F 0 "#PWR0125" H 9000 5400 50  0001 C CNN
 F 1 "GND" V 9005 5522 50  0000 R CNN
 F 2 "" H 9000 5650 50  0001 C CNN
@@
 $EndComp
 $Comp
-L Jumper:SolderJumper_2_Open JP?
+L Jumper:SolderJumper_2_Open JP2
 U 1 1 61D151D0
 P 6050 7350
-F 0 "JP?" H 6050 7555 50  0000 C CNN
+F 0 "JP2" H 6050 7555 50  0000 C CNN
 F 1 "PV EN" H 6050 7464 50  0000 C CNN
 F 2 "Jumper:SolderJumper-2_P1.3mm_Open_RoundedPad1.0x1.5mm" H 6050 7350 50  0001 C CNN
@@
 $EndComp
 $Comp
-L power:+3.3V #PWR?
+L power:+3.3V #PWR0126
 U 1 1 61DB635A
 P 9000 5850
-F 0 "#PWR?" H 9000 5700 50  0001 C CNN
+F 0 "#PWR0126" H 9000 5700 50  0001 C CNN
 F 1 "+3.3V" V 9015 5978 50  0000 L CNN
 F 2 "" H 9000 5850 50  0001 C CNN
@@
 $EndComp
 $Comp
-L power:+3.3V #PWR?
+L power:+3.3V #PWR0127
 U 1 1 61DB712B
 P 6200 6550
-F 0 "#PWR?" H 6200 6400 50  0001 C CNN
+F 0 "#PWR0127" H 6200 6400 50  0001 C CNN
 F 1 "+3.3V" V 6215 6678 50  0000 L CNN
 F 2 "" H 6200 6550 50  0001 C CNN
@@
 	9200 7950 9000 7950
 $Comp
-L Device:C_Small C?
+L Device:C_Small C57
 U 1 1 61DD3D8B
 P 9300 6000
-F 0 "C?" H 9392 6046 50  0000 L CNN
+F 0 "C57" H 9392 6046 50  0000 L CNN
 F 1 "_" H 9392 5955 50  0000 L CNN
 F 2 "Capacitor_SMD:C_0402_1005Metric" H 9300 6000 50  0001 C CNN
@@
 Connection ~ 9200 6000
 $Comp
-L power:GND #PWR?
+L power:GND #PWR0128
 U 1 1 61E003BA
 P 9400 6000
-F 0 "#PWR?" H 9400 5750 50  0001 C CNN
+F 0 "#PWR0128" H 9400 5750 50  0001 C CNN
 F 1 "GND" V 9405 5872 50  0000 R CNN
 F 2 "" H 9400 6000 50  0001 C CNN
@@
 $EndComp
 $Comp
-L power:+3.3V #PWR?
+L power:+3.3V #PWR0129
 U 1 1 61E01CF3
 P 9000 6050
-F 0 "#PWR?" H 9000 5900 50  0001 C CNN
+F 0 "#PWR0129" H 9000 5900 50  0001 C CNN
 F 1 "+3.3V" V 9015 6178 50  0000 L CNN
 F 2 "" H 9000 6050 50  0001 C CNN
@@
 $EndComp
 $Comp
-L power:+3.3V #PWR?
+L power:+3.3V #PWR0130
 U 1 1 61E10769
 P 9000 6350
-F 0 "#PWR?" H 9000 6200 50  0001 C CNN
+F 0 "#PWR0130" H 9000 6200 50  0001 C CNN
 F 1 "+3.3V" V 9015 6478 50  0000 L CNN
 F 2 "" H 9000 6350 50  0001 C CNN
@@
 $EndComp
 $Comp
-L power:+3.3V #PWR?
+L power:+3.3V #PWR0131
 U 1 1 61E1F0DC
 P 9000 6750
-F 0 "#PWR?" H 9000 6600 50  0001 C CNN
+F 0 "#PWR0131" H 9000 6600 50  0001 C CNN
 F 1 "+3.3V" V 9015 6878 50  0000 L CNN
 F 2 "" H 9000 6750 50  0001 C CNN
@@
 $EndComp
 $Comp
-L power:+3.3V #PWR?
+L power:+3.3V #PWR0132
 U 1 1 61E2DB74
 P 9000 7650
-F 0 "#PWR?" H 9000 7500 50  0001 C CNN
+F 0 "#PWR0132" H 9000 7500 50  0001 C CNN
 F 1 "+3.3V" V 9015 7778 50  0000 L CNN
 F 2 "" H 9000 7650 50  0001 C CNN

Commit message: ditch LoRa, switch processor to STM32WB30CE
Parts:
- removed C27, C28, C29, C30, C31, C32, C33, C34, C35: 0.1uF, Capacitor_SMD:C_0402_1005Metric, symbol Device:C_Small
- removed C37, C38, C39, C40, C41, C42, C43, C44, C45, C46, C47, C48, C49, C50, C51, C52, C57: _, Capacitor_SMD:C_0402_1005Metric, symbol Device:C_Small
- removed J5: RX, Connector_Coaxial:U.FL_Hirose_U.FL-R-SMT-1_Vertical, symbol Connector:Conn_Coaxial
- removed J7: Conn_Coaxial, Connector_Coaxial:U.FL_Hirose_U.FL-R-SMT-1_Vertical, symbol Connector:Conn_Coaxial
- removed L10, L11, L12: _, Inductor_SMD:L_0402_1005Metric, symbol pspice:INDUCTOR
- removed L3, L4, L5, L6, L7, L8, L9: 1uH, Inductor_SMD:L_0402_1005Metric, symbol pspice:INDUCTOR
- removed TP12: RX, TestPoint:TestPoint_Pad_2.0x2.0mm, symbol Connector:TestPoint
- removed TP13: TX, TestPoint:TestPoint_Pad_2.0x2.0mm, symbol Connector:TestPoint
- removed TP15: BLE RSTN, TestPoint:TestPoint_Pad_2.0x2.0mm, symbol Connector:TestPoint
- removed TP8: JTMS-SWDIO, TestPoint:TestPoint_Pad_2.0x2.0mm, symbol Connector:TestPoint
- removed TP9: JTO-SWCLK, TestPoint:TestPoint_Pad_2.0x2.0mm, symbol Connector:TestPoint
- removed U1: BLUENRG-355MC, libs:BLUENRG, symbol BLUENRG:BLUENRG-355MC
- removed U3: STM32WL55CCU7, libs:STM32WL55CCU7, symbol STM32WL55CCU7:STM32WL55CCU7
- removed Y3, Y4: Crystal, Crystal:Crystal_SMD_2012-2Pin_2.0x1.2mm, symbol Device:Crystal
- added JP3: WP3, Jumper:SolderJumper-2_P1.3mm_Open_Pad1.0x1.5mm, symbol Jumper:SolderJumper_2_Open
- added JP4: WP2, Jumper:SolderJumper-2_P1.3mm_Open_Pad1.0x1.5mm, symbol Jumper:SolderJumper_2_Open
- added JP5: WP4, Jumper:SolderJumper-2_P1.3mm_Open_Pad1.0x1.5mm, symbol Jumper:SolderJumper_2_Open
- added U1: STM32WB30CEU5A, libs:STM32WB30CEU5A, symbol STM32WB30CEU5A:STM32WB30CEU5A
- added U3: DLF162500LT-5028A1, libs:DLF162500LT, symbol DLF162500LT:DLF162500LT-5028A1
- added U6, U7, U8, U9: CAT24M01Y, Package_SO:TSSOP-8_4.4x3mm_P0.65mm, symbol Memory_EEPROM:CAT24M01Y
- added U?: LPS25HB, Package_LGA:ST_HLGA-10_2.5x2.5mm_P0.6mm_LayoutBorder3x2y, symbol Sensor_Pressure:LPS25HB
- C21, C22: value 0.1uF -> Loading
- C23: value 0.1uF -> 1pF
- C24: value 0.1uF -> 10pF
- C25: value 0.1uF -> 100pF
- C26: value 0.1uF -> 1mF
- D2: footprint (none) -> Diode_SMD:D_0402_1005Metric
- J4: value RX -> Conn_Coaxial
- JP2: value PV EN -> WP1; footprint Jumper:SolderJumper-2_P1.3mm_Open_RoundedPad1.0x1.5mm -> Jumper:SolderJumper-2_P1.3mm_Open_Pad1.0x1.5mm
- TP1: value NRST -> TestPoint; footprint TestPoint:TestPoint_Pad_2.0x2.0mm -> TestPoint:TestPoint_Pad_1.0x1.0mm
- TP10, TP11, TP14: footprint TestPoint:TestPoint_Pad_2.0x2.0mm -> TestPoint:TestPoint_Pad_1.0x1.0mm
- TP2: value JTRST -> JTMS_SWDIO; footprint TestPoint:TestPoint_Pad_2.0x2.0mm -> TestPoint:TestPoint_Pad_1.0x1.0mm
- TP3: value BLE TX -> JTCK_SWCLK; footprint TestPoint:TestPoint_Pad_2.0x2.0mm -> TestPoint:TestPoint_Pad_1.0x1.0mm
- TP4: value JTO-SWO -> JTDI; footprint TestPoint:TestPoint_Pad_2.0x2.0mm -> TestPoint:TestPoint_Pad_1.0x1.0mm
- TP5: value PA10 -> JTDO; footprint TestPoint:TestPoint_Pad_2.0x2.0mm -> TestPoint:TestPoint_Pad_1.0x1.0mm
- TP6: value BLE RX -> NJTRST; footprint TestPoint:TestPoint_Pad_2.0x2.0mm -> TestPoint:TestPoint_Pad_1.0x1.0mm
- TP7: value JTCK-SWDIO -> BOOT0; footprint TestPoint:TestPoint_Pad_2.0x2.0mm -> TestPoint:TestPoint_Pad_1.0x1.0mm
- Y1: value Crystal -> 32 kHz
- Y2: value Crystal -> 32 MHz
Connections:
- net RX1 is gone; now on net RX: IC2.2 (TX)
- net TX1 is gone; now on net TX: IC2.3 (RX)
- net +3V3: now also C23.1, C24.1, C25.1, C26.1, JP2.2 (B), JP3.2 (B), JP4.2 (B), JP5.2 (B), U1.1 (VBAT), U1.20 (VDD), U1.23 (VDDRF), U1.31 (VDD), U1.33 (VDD), U1.34 (VDD), U1.35 (VDD), U1.40 (VDD), U1.48 (VDD), U1.8 (VDDA), U6.2 (A1), U6.3 (A2), U6.8 (VCC), U7.8 (VCC), U8.2 (A1), U8.8 (VCC), U9.3 (A2), U9.8 (VCC)
- net GND: now also C24.2, C26.2, U1.22 (VSSRF), U1.32 (VSS), U1.49 (VSS), U3.2 (GND), U3.4 (GND), U6.4 (GND), U7.2 (A1), U7.3 (A2), U7.4 (GND), U8.3 (A2), U8.4 (GND), U9.2 (A1), U9.4 (GND)
- net RX: now also U1.36 (PA10)
- net SCL: now also U1.5 (PB8), U6.6 (SCL), U7.6 (SCL), U8.6 (SCL), U9.6 (SCL)
- net SDA: now also U1.6 (PB9), U6.5 (SDA), U7.5 (SDA), U8.5 (SDA), U9.5 (SDA)
- net SPI1-MOSI: now also U1.16 (PA7)
- net SPI1-SCK: now also U1.10 (PA1)
- net TX: now also U1.18 (PA9)
- net at BT1.1 (+), C53.1, JP1.2 (B)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: now also U1.9 (PA0)
- net at IC2.4 (1PPS): now also U1.11 (PA2)
- net at IC2.5 (WAKE-UP): now also U1.12 (PA3)
- net at TP4.1: now also U1.42 (PA15(JTDI))
- net at J3.5 (Pin_5): now also U1.28 (PB0)
- net at TP1.1: now also U1.7 (NRST)
- net at TP2.1: now also U1.39 (PA13(JTMS_SWDIO))
- net at Y1.2: now also C22.1, U1.3 (PC15-OSC32_OUT)
- net at Y1.1: now also C21.1, U1.2 (PC14-OSC32_IN)
- net at R4.1, SW2.1: now also U1.46 (PB6)
- net at J3.6 (Pin_6): now also U1.29 (PB1)
- net at R3.1, SW1.1: now also U1.47 (PB7)
- net at R5.1, SW3.1: now also U1.45 (PB5)
- net at Y2.2: now also U1.24 (OSC_OUT)
- net at Y2.1: now also U1.25 (OSC_IN)
- net at TP7.1: now also U1.4 (PH3-BOOT0)
- net at J3.7 (Pin_7): now also U1.19 (PB2)
- net at J3.8 (Pin_8): now also U1.17 (PA8)
- net at J3.9 (Pin_9): now also U1.15 (PA6)
- net at J4.1 (In): now also U3.3 (OUT)
- net at TP5.1: now also U1.43 (PB3(JTDO))
- net at TP3.1: now also U1.41 (PA14(JTCK_SWCLK))
- net at TP6.1: now also U1.44 (PB4(NJTRST))
- net at JP2.1 (A): now also U6.7 (WP)
- removed net VR_PA: C21.1, C22.1
- new net: U1.21 (RF1), U3.1 (IN)
- new net: JP4.1 (A), U8.7 (WP)
- new net: JP3.1 (A), U7.7 (WP)
- new net: JP5.1 (A), U9.7 (WP)
- new net: U?.3 (GND), U?.8 (GND), U?.9 (GND)
Other:
- note removed: "BLE\n\n"
- note removed: "LoRa RF\n"
- moved on the sheet: D2, IC1, IC2, J2, R3, R4, R5, SW1, SW2, SW3
