File: MainBoard/MainBoard.sch (KiCad schematic (older format))
At the start: 80 parts, among them IC1 MAX30102, IC2 TESEO-LIV3F, J1 PV IN, J2 Conn_Coaxial, J3 Conn_01x30_Female, J4 Conn_Coaxial, J6 Conn_01x04, SW1 SW_DIP_x01, SW2 SW_DIP_x01, SW3 SW_DIP_x01, U1 STM32WB30CEU5A, U2 MAX20361AEWC+, U3 DLF162500LT-5028A1, U4 LSM9DS1, U5 TPS63001, U6 CAT24M01Y, U7 CAT24M01Y, U8 CAT24M01Y, U9 CAT24M01Y, Y1 32 kHz, Y2 32 MHz

Commit message: route entire damn thing in one sitting
Parts:
- removed U?: LPS25HB, Package_LGA:ST_HLGA-10_2.5x2.5mm_P0.6mm_LayoutBorder3x2y, symbol Sensor_Pressure:LPS25HB
Other:
- moved on the sheet: D2, IC1
Changed lines of the file:
@@
 L Sensor:MAX30102 IC1
 U 1 1 605E8DCD
-P 4100 5300
-F 0 "IC1" H 3456 5346 50  0000 R CNN
-F 1 "MAX30102" H 3456 5255 50  0000 R CNN
-F 2 "OptoDevice:Maxim_OLGA-14_3.3x5.6mm_P0.8mm" H 3950 6200 50  0001 C CNN
-F 3 "https://datasheets.maximintegrated.com/en/ds/MAX30102.pdf" H 3750 5550 50  0001 C CNN
-	1    4100 5300
+P 3900 4200
+F 0 "IC1" H 3256 4246 50  0000 R CNN
+F 1 "MAX30102" H 3256 4155 50  0000 R CNN
+F 2 "OptoDevice:Maxim_OLGA-14_3.3x5.6mm_P0.8mm" H 3750 5100 50  0001 C CNN
+F 3 "https://datasheets.maximintegrated.com/en/ds/MAX30102.pdf" H 3550 4450 50  0001 C CNN
+	1    3900 4200
 	1    0    0    -1
 $EndComp
@@
 Text GLabel 900  4350 0    50   Input ~ 0
 SDA
-Text GLabel 3500 5200 1    50   Input ~ 0
+Text GLabel 3300 4100 1    50   Input ~ 0
 SCL
-Text GLabel 3500 5300 3    50   Input ~ 0
+Text GLabel 3300 4200 3    50   Input ~ 0
 SDA
 $Comp
@@
 L power:GND #PWR0110
 U 1 1 60603461
-P 4200 5800
-F 0 "#PWR0110" H 4200 5550 50  0001 C CNN
-F 1 "GND" H 4205 5627 50  0000 C CNN
-F 2 "" H 4200 5800 50  0001 C CNN
-F 3 "" H 4200 5800 50  0001 C CNN
-	1    4200 5800
+P 4000 4700
+F 0 "#PWR0110" H 4000 4450 50  0001 C CNN
+F 1 "GND" H 4005 4527 50  0000 C CNN
+F 2 "" H 4000 4700 50  0001 C CNN
+F 3 "" H 4000 4700 50  0001 C CNN
+	1    4000 4700
 	0    -1   -1   0
 $EndComp
@@
 L power:GND #PWR0111
 U 1 1 60603AAF
-P 4000 5800
-F 0 "#PWR0111" H 4000 5550 50  0001 C CNN
-F 1 "GND" H 4005 5627 50  0000 C CNN
-F 2 "" H 4000 5800 50  0001 C CNN
-F 3 "" H 4000 5800 50  0001 C CNN
-	1    4000 5800
+P 3800 4700
+F 0 "#PWR0111" H 3800 4450 50  0001 C CNN
+F 1 "GND" H 3805 4527 50  0000 C CNN
+F 2 "" H 3800 4700 50  0001 C CNN
+F 3 "" H 3800 4700 50  0001 C CNN
+	1    3800 4700
 	1    0    0    -1
 $EndComp
@@
 Text Notes 10950 4544 2    197  ~ 0
 LoRa + main uC\n
-Text Notes 5100 5044 2    197  ~ 0
+Text Notes 4900 3944 2    197  ~ 0
 HR
 Text Notes 1450 3844 2    197  ~ 0
@@
 L Device:D_Zener D2
 U 1 1 61699C7D
-P 3650 4800
-F 0 "D2" V 3604 4880 50  0000 L CNN
-F 1 "1.8V" V 3695 4880 50  0000 L CNN
-F 2 "Diode_SMD:D_0402_1005Metric" H 3650 4800 50  0001 C CNN
-F 3 "~" H 3650 4800 50  0001 C CNN
-	1    3650 4800
+P 3450 3700
+F 0 "D2" V 3404 3780 50  0000 L CNN
+F 1 "1.8V" V 3495 3780 50  0000 L CNN
+F 2 "Diode_SMD:D_0402_1005Metric" H 3450 3700 50  0001 C CNN
+F 3 "~" H 3450 3700 50  0001 C CNN
+	1    3450 3700
 	1    0    0    -1
 $EndComp
@@
 L power:+3.3V #PWR0101
 U 1 1 616B07A5
-P 3500 4800
-F 0 "#PWR0101" H 3500 4650 50  0001 C CNN
-F 1 "+3.3V" V 3515 4928 50  0000 L CNN
-F 2 "" H 3500 4800 50  0001 C CNN
-F 3 "" H 3500 4800 50  0001 C CNN
-	1    3500 4800
+P 3300 3700
+F 0 "#PWR0101" H 3300 3550 50  0001 C CNN
+F 1 "+3.3V" V 3315 3828 50  0000 L CNN
+F 2 "" H 3300 3700 50  0001 C CNN
+F 3 "" H 3300 3700 50  0001 C CNN
+	1    3300 3700
 	0    -1   -1   0
 $EndComp
@@
 L power:+3.3V #PWR0102
 U 1 1 616B2A6C
-P 4000 4800
-F 0 "#PWR0102" H 4000 4650 50  0001 C CNN
-F 1 "+3.3V" H 4015 4973 50  0000 C CNN
-F 2 "" H 4000 4800 50  0001 C CNN
-F 3 "" H 4000 4800 50  0001 C CNN
-	1    4000 4800
-	1    0    0    -1
-$EndComp
-Wire Wire Line
-	4000 4800 4100 4800
-Connection ~ 4000 4800
+P 3800 3700
+F 0 "#PWR0102" H 3800 3550 50  0001 C CNN
+F 1 "+3.3V" H 3815 3873 50  0000 C CNN
+F 2 "" H 3800 3700 50  0001 C CNN
+F 3 "" H 3800 3700 50  0001 C CNN
+	1    3800 3700
+	1    0    0    -1
+$EndComp
+Wire Wire Line
+	3800 3700 3900 3700
+Connection ~ 3800 3700
 $Comp
 L Regulator_Switching:TPS63001 U5
@@
 	1    0    0    -1
 $EndComp
-$Comp
-L Sensor_Pressure:LPS25HB U?
-U 1 1 60864EE9
-P 2250 9250
-F 0 "U?" H 1820 9246 50  0000 R CNN
-F 1 "LPS25HB" H 1820 9155 50  0000 R CNN
-F 2 "Package_LGA:ST_HLGA-10_2.5x2.5mm_P0.6mm_LayoutBorder3x2y" H 2250 9050 50  0001 C CNN
-F 3 "www.st.com/resource/en/datasheet/lps25hb.pdf" H 2300 8900 50  0001 C CNN
-	1    2250 9250
-	1    0    0    -1
-$EndComp
