File: MainBoard/MainBoard.sch (KiCad schematic (older format))
At the start: 59 parts, among them IC1 MAX30102, J3 Conn_01x30_Female, J6 Conn_01x04, SW1 SW_DIP_x01, SW2 SW_DIP_x01, SW3 SW_DIP_x01, U1 ESP32-WROOM-32, U2 ADP2108AUJ-3.3, U3 LSM303C

Commit message: switch processor, add sensors, change shape'
Parts:
- removed BZ1: Buzzer, libs:PB9.11-5v, symbol Device:Buzzer
- removed J6: Conn_01x04, libs:4 Pin SMD Wire, symbol Connector_Generic:Conn_01x04
- removed JP1: WP, Jumper:SolderJumper-2_P1.3mm_Open_Pad1.0x1.5mm, symbol Jumper:SolderJumper_2_Open
- removed L1: 1uH, Inductor_SMD:L_0805_2012Metric, symbol Device:L_Small
- removed R2, R6, R7, R8: 2k, Resistor_SMD:R_0402_1005Metric, symbol Device:R_US
- removed TP11: BATT, TestPoint:TestPoint_Pad_1.0x1.0mm, symbol Connector:TestPoint
- removed TP8: STX, TestPoint:TestPoint_Pad_1.0x1.0mm, symbol Connector:TestPoint
- removed TP9: SRX, TestPoint:TestPoint_Pad_1.0x1.0mm, symbol Connector:TestPoint
- removed U1: ESP32-WROOM-32, RF_Module:ESP32-WROOM-32, symbol RF_Module:ESP32-WROOM-32
- removed U2: ADP2108AUJ-3.3, Package_TO_SOT_SMD:TSOT-23-5, symbol Regulator_Switching:ADP2108AUJ-3.3
- added AE1: ACAG0301-1575-T, libs:ANT-ACAG0301-1575-T, symbol ACAG0301-1575-T:ACAG0301-1575-T
- added C21: 22pF, Capacitor_SMD:C_0402_1005Metric, symbol Device:C_Small
- added D3: LED, LED_SMD:LED_0402_1005Metric, symbol Device:LED
- added D4: MBR120, Diode_SMD:D_SOD-123F, symbol Diode:MBR1020VL
- added IC2: TESEO-LIV3F, libs:SON110P970X1010X230-18N, symbol TESEO-LIV3F:TESEO-LIV3F
- added J1: USB_C_Receptacle_USB2.0, Connector_USB:USB_C_Receptacle_GCT_USB4085, symbol Connector:USB_C_Receptacle_USB2.0
- added J2: Micro_SD_Card, Connector_Card:microSD_HC_Molex_104031-0811, symbol Connector:Micro_SD_Card
- added L1: 10uH, Inductor_SMD:L_0402_1005Metric, symbol Device:L
- added Q1: DMG2301L, Package_TO_SOT_SMD:SOT-23, symbol Transistor_FET:DMG2301L
- added R10, R11, R12, R9: 100k, Resistor_SMD:R_0402_1005Metric, symbol Device:R_Small_US
- added R13, R14: 56k, Resistor_SMD:R_0402_1005Metric, symbol Device:R_Small_US
- added R2, R6: 5.7k, Resistor_SMD:R_0402_1005Metric, symbol Device:R_Small_US
- added R7: 4.7k, Resistor_SMD:R_0402_1005Metric, symbol Device:R_Small_US
- added R8: 1k, Resistor_SMD:R_0402_1005Metric, symbol Device:R_Small_US
- added U1: MCP73831-2-OT, Package_TO_SOT_SMD:SOT-23-5, symbol Battery_Management:MCP73831-2-OT
- added U2: MDBT50Q-1MV2, libs:XCVR_MDBT50Q-1MV2, symbol MDBT50Q-1MV2:MDBT50Q-1MV2
- added U4: AP2112K-3.3, Package_TO_SOT_SMD:SOT-23-5, symbol Regulator_Linear:AP2112K-3.3
- added U5: VL53L1CXV0FY1, Sensor_Distance:ST_VL53L1x, symbol Sensor_Distance:VL53L1CXV0FY1
- added U6: MPL3115A2, Package_LGA:NXP_LGA-8_3x5mm_P1.25mm_H1.1mm, symbol Sensor_Pressure:MPL3115A2
- added U7: Si7050-A20, Package_DFN_QFN:DFN-6-1EP_3x3mm_P1mm_EP1.5x2.4mm, symbol Sensor_Temperature:Si7050-A20
- added Y1: ABS05W, Crystal:Crystal_SMD_MicroCrystal_CM9V-T1A-2Pin_1.6x1.0mm, symbol Device:Crystal
- BT1: footprint Connector_PinHeader_1.00mm:PinHeader_1x02_P1.00mm_Vertical -> Connector_PinHeader_1.27mm:PinHeader_1x02_P1.27mm_Vertical_SMD_Pin1Left
- C1: value 4.5uF -> 10uF
- C2: value 5.7k -> 10uF
- C3: value 5.7k -> 22pF
- TP1: value RST -> nRFRESET; footprint TestPoint:TestPoint_Pad_1.0x1.0mm -> TestPoint:TestPoint_Pad_2.0x2.0mm
- TP10, TP14: footprint TestPoint:TestPoint_Pad_1.0x1.0mm -> TestPoint:TestPoint_Pad_2.0x2.0mm
- TP2: value IO12 -> GPSRESET; footprint TestPoint:TestPoint_Pad_1.0x1.0mm -> TestPoint:TestPoint_Pad_2.0x2.0mm
- TP3: value IO14 -> SWDIO; footprint TestPoint:TestPoint_Pad_1.0x1.0mm -> TestPoint:TestPoint_Pad_2.0x2.0mm
- TP4: value BOOT0 -> SW0; footprint TestPoint:TestPoint_Pad_1.0x1.0mm -> TestPoint:TestPoint_Pad_2.0x2.0mm
- TP5: value IO13 -> SWCLK; footprint TestPoint:TestPoint_Pad_1.0x1.0mm -> TestPoint:TestPoint_Pad_2.0x2.0mm
- TP6: value IO15 -> SDA; footprint TestPoint:TestPoint_Pad_1.0x1.0mm -> TestPoint:TestPoint_Pad_2.0x2.0mm
- TP7: value BOOT1 -> SCL; footprint TestPoint:TestPoint_Pad_1.0x1.0mm -> TestPoint:TestPoint_Pad_2.0x2.0mm
Connections:
- net labels added: RXD, TXD
- wire segments 95 -> 135
Other:
- moved on the sheet: C10, C11, C12, C13, C14, C15, C16, C17, C18, C19, C20, C23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

Commit message: update pdf's
Parts:
- added C22: 100nF, Capacitor_SMD:C_0402_1005Metric, symbol MainBoard-rescue:C_Small-Device
- added D5: LED, LED_SMD:LED_Kingbright_APFA3010_3x1.5mm_Horizontal, symbol Device:LED
- added R15: 1K, Resistor_SMD:R_0402_1005Metric, symbol MainBoard-rescue:R_Small_US-Device
- BT1: symbol Device:Battery_Cell -> MainBoard-rescue:Battery_Cell-Device
- C1, C10, C11, C12, C13, C14, C15, C16, C17, C18, C19, C2, C20, C21, C23, C24, C25, C26, C3, C4, C5, C6, C7, C8, C9: symbol Device:C_Small -> MainBoard-rescue:C_Small-Device
- D1: symbol pspice:DIODE -> MainBoard-rescue:DIODE-pspice
- D2: symbol Device:D_Zener -> MainBoard-rescue:D_Zener-Device
- D3: symbol Device:LED -> MainBoard-rescue:LED-Device
- D4: symbol Diode:MBR1020VL -> MainBoard-rescue:MBR1020VL-Diode
- IC1: symbol Sensor:MAX30102 -> MainBoard-rescue:MAX30102-Sensor
- J1: symbol Connector:USB_C_Receptacle_USB2.0 -> MainBoard-rescue:USB_C_Receptacle_USB2.0-Connector
- J2: symbol Connector:Micro_SD_Card -> MainBoard-rescue:Micro_SD_Card-Connector
- J3: symbol Connector:Conn_01x30_Female -> MainBoard-rescue:Conn_01x30_Female-Connector
- L1: symbol Device:L -> MainBoard-rescue:L-Device
- Q1: symbol Transistor_FET:DMG2301L -> MainBoard-rescue:DMG2301L-Transistor_FET
- R1, R3, R4, R5: symbol Device:R_US -> MainBoard-rescue:R_US-Device
- R10, R11, R12, R13, R14, R2, R6, R7, R8, R9: symbol Device:R_Small_US -> MainBoard-rescue:R_Small_US-Device
- SW1, SW2, SW3: symbol Switch:SW_DIP_x01 -> MainBoard-rescue:SW_DIP_x01-Switch
- TP1, TP10, TP14, TP2, TP3, TP4, TP5, TP6, TP7: symbol Connector:TestPoint -> MainBoard-rescue:TestPoint-Connector
- U1: symbol Battery_Management:MCP73831-2-OT -> MainBoard-rescue:MCP73831-2-OT-Battery_Management
- U3: symbol Sensor_Motion:LSM303C -> MainBoard-rescue:LSM303C-Sensor_Motion
- U4: symbol Regulator_Linear:AP2112K-3.3 -> MainBoard-rescue:AP2112K-3.3-Regulator_Linear
- U5: symbol Sensor_Distance:VL53L1CXV0FY1 -> MainBoard-rescue:VL53L1CXV0FY1-Sensor_Distance
- U6: symbol Sensor_Pressure:MPL3115A2 -> MainBoard-rescue:MPL3115A2-Sensor_Pressure
- U7: symbol Sensor_Temperature:Si7050-A20 -> MainBoard-rescue:Si7050-A20-Sensor_Temperature
- Y1: symbol Device:Crystal -> MainBoard-rescue:Crystal-Device
Connections:
- wire segments 135 -> 169
Other:
- moved on the sheet: C10, C11, C12, C13, C14, C15, C16, C17, C18, C19, C20, C5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

Commit message: oops! I forgot the buzzer
Parts:
- added BZ1: Buzzer, libs:PB9.11-5v, symbol Device:Buzzer
- added R16: JUST IN CASE, Resistor_SMD:R_0402_1005Metric, symbol MainBoard-rescue:R_Small_US-Device
Connections:
- net GND: now also R16.1
- net at U2.24 (P0.08): now also BZ1.1 (-)
- new net: BZ1.2 (+), R16.2
Changed lines of the file:
@@
 Wire Wire Line
 	10700 5750 10750 5750
+Wire Wire Line
+	6600 6200 6300 6200
+Wire Wire Line
+	6300 6200 6300 6350
+Wire Wire Line
+	6300 6350 4100 6350
+$Comp
+L Device:Buzzer BZ1
+U 1 1 60B842BC
+P 4000 6250
+F 0 "BZ1" H 4005 5925 50  0000 C CNN
+F 1 "Buzzer" H 4005 6016 50  0000 C CNN
+F 2 "libs:PB9.11-5v" V 3975 6350 50  0001 C CNN
+F 3 "~" V 3975 6350 50  0001 C CNN
+	1    4000 6250
+	-1   0    0    1
+$EndComp
+$Comp
+L power:GND #PWR0146
+U 1 1 60B855FB
+P 4300 6150
+F 0 "#PWR0146" H 4300 5900 50  0001 C CNN
+F 1 "GND" V 4305 6022 50  0000 R CNN
+F 2 "" H 4300 6150 50  0001 C CNN
+F 3 "" H 4300 6150 50  0001 C CNN
+	1    4300 6150
+	0    -1   -1   0
+$EndComp
+$Comp
+L MainBoard-rescue:R_Small_US-Device R16
+U 1 1 60B8D5FB
+P 4200 6150
+F 0 "R16" H 4268 6196 50  0000 L CNN
+F 1 "JUST IN CASE" H 4268 6105 50  0000 L CNN
+F 2 "Resistor_SMD:R_0402_1005Metric" H 4200 6150 50  0001 C CNN
+F 3 "~" H 4200 6150 50  0001 C CNN
+	1    4200 6150
+	0    1    1    0
+$EndComp
 $EndSCHEMATC

Commit message: route board
Parts:
- added TP8: NFC1, TestPoint:TestPoint_Pad_2.0x2.0mm, symbol MainBoard-rescue:TestPoint-Connector
- added TP9: NFC2, TestPoint:TestPoint_Pad_2.0x2.0mm, symbol MainBoard-rescue:TestPoint-Connector
Connections:
- net at U2.52 (P0.09/NFC1): now also TP8.1
- net at U2.54 (P0.10/NFC2): now also TP9.1
Changed lines of the file:
@@
 	0    1    1    0
 $EndComp
+$Comp
+L MainBoard-rescue:TestPoint-Connector TP8
+U 1 1 60BAC43F
+P 6600 6300
+F 0 "TP8" V 6795 6372 50  0000 C CNN
+F 1 "NFC1" V 6704 6372 50  0000 C CNN
+F 2 "TestPoint:TestPoint_Pad_2.0x2.0mm" H 6800 6300 50  0001 C CNN
+F 3 "~" H 6800 6300 50  0001 C CNN
+	1    6600 6300
+	0    -1   -1   0
+$EndComp
+$Comp
+L MainBoard-rescue:TestPoint-Connector TP9
+U 1 1 60BB7090
+P 6600 6400
+F 0 "TP9" V 6795 6472 50  0000 C CNN
+F 1 "NFC2" V 6704 6472 50  0000 C CNN
+F 2 "TestPoint:TestPoint_Pad_2.0x2.0mm" H 6800 6400 50  0001 C CNN
+F 3 "~" H 6800 6400 50  0001 C CNN
+	1    6600 6400
+	0    -1   -1   0
+$EndComp
 $EndSCHEMATC
