File: Finger Boards/FingerBoard/FingerBoard.kicad_pcb (KiCad board)
At the start: 2 copper layers, 4.8 x 6.8 mm, 7 parts, among them U1 LSM303C

Commit message: I dont even remember
Other:
- board size 4.8 x 6.8 mm -> 6.2 x 7.5 mm
Changed lines of the file:
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@@
       (outputformat 1)
       (mirror false)
-      (drillshape 1)
+      (drillshape 0)
       (scaleselection 1)
-      (outputdirectory ""))
+      (outputdirectory "Gerber/"))
   )
   (net 0 "")
@@
     )
   )
-  (gr_line (start 146.5 56.4) (end 146.5 63.2) (layer Edge.Cuts) (width 0.05))
-  (gr_line (start 151.3 56.4) (end 146.5 56.4) (layer Edge.Cuts) (width 0.05))
-  (gr_line (start 151.3 63.2) (end 151.3 56.4) (layer Edge.Cuts) (width 0.05))
-  (gr_line (start 146.5 63.2) (end 151.3 63.2) (layer Edge.Cuts) (width 0.05))
+  (gr_line (start 145.75 56) (end 145.75 63.5) (layer Edge.Cuts) (width 0.1))
+  (gr_line (start 152 56) (end 145.75 56) (layer Edge.Cuts) (width 0.1))
+  (gr_line (start 152 63.5) (end 152 56) (layer Edge.Cuts) (width 0.1))
+  (gr_line (start 145.75 63.5) (end 152 63.5) (layer Edge.Cuts) (width 0.1))
   (segment (start 147.23 59.55) (end 148.1375 59.55) (width 0.15) (layer F.Cu) (net 1))
   (segment (start 147 59.32) (end 147.23 59.55) (width 0.15) (layer F.Cu) (net 1))
@@
     (polygon
       (pts
-        (xy 146.4 56.3) (xy 146.4 63.3) (xy 151.4 63.3) (xy 151.4 56.3)
+        (xy 145.75 56) (xy 145.75 63.5) (xy 152 63.5) (xy 152 56)
       )
     )
