File: Band/Band.kicad_sch (KiCad schematic)
At the start: 15 parts

Commit message: finish schematic
Parts:
- added R3, R4: 1k, Resistor_SMD:R_0402_1005Metric, symbol Device:R_Small_US
- added TP5: RX, TestPoint:TestPoint_Pad_2.0x2.0mm, symbol Connector:TestPoint
- added TP7: TX, TestPoint:TestPoint_Pad_2.0x2.0mm, symbol Connector:TestPoint
- added U2: TC2014-1.8VxCTTR, Package_TO_SOT_SMD:SOT-23-5, symbol Regulator_Linear:TC2014-1.8VxCTTR
- R1, R2: renamed from R?; footprint (none) -> Resistor_SMD:R_0402_1005Metric
- TP1, TP10, TP2, TP3, TP4, TP6, TP8, TP9: renamed from TP?; footprint (none) -> TestPoint:TestPoint_Pad_2.0x2.0mm
- U4: renamed from U?; footprint XDCR_BMI270 -> BMI270:XDCR_BMI270
- gave numbers to parts that had none: 4
Connections:
- net +3.3V: now also U1.2 (EN/CHIP_PU), U5.10 (VLED+), U5.9 (VLED+), U2.1 (VIN)
- net GND: now also U3.1 (GND), U3.7 (GND), U5.4 (PGND), R3.1, U2.2 (GND)
- net Power_Management/BATT: now also R4.2
- net SCL: now also U1.8 (GPIO9)
- net SDA: now also U1.10 (GPIO10)
- net at U1.11 (GPIO20/U0RXD): now also TP5.1
- net at U1.12 (GPIO21/U0TXD): now also TP7.1
- net at U1.15 (GPIO3/ADC1_CH3): now also U4.9 (INT2)
- net SPI_MISO: now reaches U1.16 (GPIO2/ADC1_CH2)
- net SPI_MISO: now also U3.5 (SDO)
- net at U1.18 (GPIO0/ADC1_CH0/XTAL_32K_P): now also R3.2, R4.1
- net at U1.3 (GPIO4/ADC1_CH4): now also U4.4 (INT1)
- net at U1.4 (GPIO5/ADC2_CH0): now also U3.2 (CSB)
- net SPI_SCK: now reaches U1.5 (GPIO6)
- net SPI_SCK: now also U3.4 (SCK)
- net SPI_MOSI: now reaches U1.6 (GPIO7)
- net SPI_MOSI: now also U3.3 (SDI)
- net at U1.7 (GPIO8): now also U2.3 (ON/~{OFF})
- net at U5.11 (VDD): now also U3.6 (VDDIO), U3.8 (VDD), U2.5 (VOUT)

Commit message: preliminary layout
Parts:
- removed J1: USB_C_Receptacle_USB2.0, symbol Connector:USB_C_Receptacle_USB2.0
- removed R1, R2: 5.1k, Resistor_SMD:R_0402_1005Metric, symbol Device:R_Small_US
- removed TP10: BATT, TestPoint:TestPoint_Pad_2.0x2.0mm, symbol Connector:TestPoint
- removed TP4: PV, TestPoint:TestPoint_Pad_2.0x2.0mm, symbol Connector:TestPoint
- removed TP9: GND, TestPoint:TestPoint_Pad_2.0x2.0mm, symbol Connector:TestPoint
- added TP11: D-, TestPoint:TestPoint_Pad_2.0x2.0mm, symbol Connector:TestPoint
- added TP12: D+, TestPoint:TestPoint_Pad_2.0x2.0mm, symbol Connector:TestPoint
Connections:
- net at U1.14 (GPIO19/USB_D+): now also TP12.1
- net at U1.13 (GPIO18/USB_D-): now also TP11.1
